Commit message: update example

File: urdf/example.urdf (robot description, URDF)
Before this commit: robot example_3dof_manipulator, 4 links, 3 joints
Joints:
- joint elbow: origin (none) -> xyz=0.2 0 0
- joint shoulder: origin (none) -> xyz=0 0 0
- joint wrist: limit effort=10.0 velocity=1.0 -> lower=-1.0 upper=1.0 effort=10.0 velocity=1.0; origin (none) -> xyz=0.2 0 0

Commit message: migrate the entire package to ROS2

File: urdf/example.urdf (robot description, URDF)
Before this commit: robot example_3dof_manipulator, 4 links, 3 joints
Links:
- link body: geometry visual box size=0.10 0.10 0.10
- link forearm: geometry visual box size=0.20 0.06 0.06
- link hand: geometry visual box size=0.04 0.04 0.04
- link upper_arm: geometry visual box size=0.20 0.08 0.08
