Commit message: give visuals to single actuator example model

File: examples/single_actuator/description/model.xacro (robot description, xacro)
@@ -1,10 +1,34 @@
 <?xml version="1.0"?>
 <robot>
-    <!-- TODO: add visual, collision, material, etc -->
-    <link name="body" />
+    <!-- TODO: add collision, etc -->
+    <link name="body">
+        <visual>
+            <geometry>
+                <box size="0.20 0.10 0.10" />
+            </geometry>
+            <material name="blue" />
+        </visual>
+    </link>
     <joint name="axis" type="continuous">
+        <origin xyz="0.10 0 0" />
         <parent link="body" />
         <child link="wheel" />
+        <axis xyz="1 0 0" />
     </joint>
-    <link name="wheel" />
+    <link name="wheel">
+        <visual>
+            <origin xyz="0.01 0 0" rpy="0 ${pi/2} 0" />
+            <geometry>
+                <cylinder radius="0.05" length="0.02" />
+            </geometry>
+            <material name="red" />
+        </visual>
+        <visual>
+            <origin xyz="0.01 0 0.05" rpy="0 0 0" />
+            <geometry>
+                <box size="0.02 0.02 0.1" />
+            </geometry>
+            <material name="red" />
+        </visual>
+    </link>
 </robot>

Commit message: set inertial param to links

File: examples/single_actuator/description/model.xacro (robot description, xacro)
@@ -1,6 +1,10 @@
 <?xml version="1.0"?>
 <robot>
-    <!-- TODO: add collision, etc -->
+    <!-- TODO: more reasonable inertial params, add collision, etc -->
     <link name="body">
+        <inertial>
+            <mass value="100" />
+            <inertia ixx="100" ixy="0" ixz="0" iyy="100" iyz="0" izz="100" />
+        </inertial>
         <visual>
             <geometry>
@@ -17,4 +21,8 @@
     </joint>
     <link name="wheel">
+        <inertial>
+            <mass value="1" />
+            <inertia ixx="1" ixy="0" ixz="0" iyy="1" iyz="0" izz="1" />
+        </inertial>
         <visual>
             <origin xyz="0.01 0 0" rpy="0 ${pi/2} 0" />
