Commit message: more organized examples

File: examples/3dof_manipulator/description/ros2_control.xacro (robot description, xacro)
@@ -1,69 +1,4 @@
-<robot name="example_3dof_manipulator">
-    <!-- body => [shoulder] => upper_arm -->
-    <link name="body">
-        <visual>
-            <geometry>
-                <box size="0.10 0.10 0.10" />
-            </geometry>
-            <material name="body_material">
-                <color rgba="0.08 0.18 0.30 1.0" />
-            </material>
-        </visual>
-    </link>
-    <joint name="shoulder" type="revolute">
-        <origin xyz="0 0 0" />
-        <parent link="body" />
-        <child link="upper_arm" />
-        <axis xyz="0 -1 0" />
-        <limit lower="0" upper="3.14" effort="10.0" velocity="1.0" />
-    </joint>
-    <link name="upper_arm">
-        <visual>
-            <origin xyz="0.1 0 0" />
-            <geometry>
-                <box size="0.20 0.08 0.08" />
-            </geometry>
-            <material name="upper_arm_material">
-                <color rgba="0.22 0.32 0.44 1.0" />
-            </material>
-        </visual>
-    </link>
-    <!-- upper_arm => [elbow] => forearm -->
-    <joint name="elbow" type="continuous">
-        <origin xyz="0.2 0 0" />
-        <parent link="upper_arm" />
-        <child link="forearm" />
-        <axis xyz="0 -1 0" />
-    </joint>
-    <link name="forearm">
-        <visual>
-            <origin xyz="0.1 0 0" />
-            <geometry>
-                <box size="0.20 0.06 0.06" />
-            </geometry>
-            <material name="forearm_material">
-                <color rgba="0.62 0.83 0.78 1.0" />
-            </material>
-        </visual>
-    </link>
-    <!-- forearm => [wrist] => hand -->
-    <joint name="wrist" type="revolute">
-        <origin xyz="0.2 0 0" />
-        <parent link="forearm" />
-        <child link="hand" />
-        <axis xyz="0 -1 0" />
-        <limit lower="-1.0" upper="1.0" effort="10.0" velocity="1.0" />
-    </joint>
-    <link name="hand">
-        <visual>
-            <geometry>
-                <box size="0.04 0.04 0.04" />
-            </geometry>
-            <material name="hand_material">
-                <color rgba="0.93 0.93 0.93 1.0" />
-            </material>
-        </visual>
-    </link>
-    <!-- -->
+<?xml version="1.0"?>
+<robot>
     <ros2_control name="LayeredHardware" type="system">
         <hardware>
@@ -106,6 +41,6 @@
                 <param name="max">6.0</param>
             </command_interface>
-            <command_interface name="effort"/>
             <state_interface name="position"/>
+            <state_interface name="velocity"/>
         </joint>
         <transmission name="shoulder_trans">
@@ -120,6 +55,6 @@
             <command_interface name="position"/>
             <command_interface name="velocity"/>
-            <command_interface name="effort"/>
             <state_interface name="position"/>
+            <state_interface name="velocity"/>
         </joint>
         <transmission name="elbow_trans">
@@ -132,7 +67,8 @@
         </transmission>
         <joint name="wrist">
-            <command_interface name="position">
-            </command_interface>
+            <command_interface name="position"/>
+            <command_interface name="velocity"/>
             <state_interface name="position"/>
+            <state_interface name="velocity"/>
         </joint>
         <transmission name="wrist_trans">

Commit message: more natural roles for transmission components

File: examples/3dof_manipulator/description/ros2_control.xacro (robot description, xacro)
@@ -46,6 +46,6 @@
         <transmission name="shoulder_trans">
             <plugin>transmission_interface/SimpleTransmission</plugin>
-            <actuator name="shoulder_actuator" role="shoulder_actuator"/>
-            <joint name="shoulder" role="shoulder">
+            <actuator name="shoulder_actuator" role="actuator"/>
+            <joint name="shoulder" role="joint">
                 <mechanical_reduction>10.0</mechanical_reduction>
                 <offset>0.0</offset>
@@ -60,6 +60,6 @@
         <transmission name="elbow_trans">
             <plugin>transmission_interface/SimpleTransmission</plugin>
-            <actuator name="elbow_actuator" role="elbow_actuator"/>
-            <joint name="elbow" role="elbow">
+            <actuator name="elbow_actuator" role="actuator"/>
+            <joint name="elbow" role="joint">
                 <mechanical_reduction>5.0</mechanical_reduction>
                 <offset>0.0</offset>
@@ -74,6 +74,6 @@
         <transmission name="wrist_trans">
             <plugin>transmission_interface/SimpleTransmission</plugin>
-            <actuator name="wrist_actuator" role="wrist_actuator"/>
-            <joint name="wrist" role="wrist">
+            <actuator name="wrist_actuator" role="actuator"/>
+            <joint name="wrist" role="joint">
                 <mechanical_reduction>2.0</mechanical_reduction>
                 <offset>0.0</offset>

File: examples/single_actuator/description/ros2_control.xacro (robot description, xacro)
@@ -40,6 +40,6 @@
         <transmission name="axis_trans">
             <plugin>transmission_interface/SimpleTransmission</plugin>
-            <actuator name="axis_actuator" role="axis_actuator"/>
-            <joint name="axis" role="axis">
+            <actuator name="axis_actuator" role="actuator"/>
+            <joint name="axis" role="joint">
                 <mechanical_reduction>10.0</mechanical_reduction>
                 <offset>0.0</offset>
